Commit message: Remove unused built-in gyro frame from Create description

File: create_description/urdf/create_base.urdf.xacro (robot description, xacro)
@@ -184,22 +184,8 @@
       <axis xyz="0 1 0" />
     </joint>
-    <joint name="gyro_joint" type="fixed">
-      <axis xyz="0 1 0" />
-      <origin xyz="0 0 0.04" rpy="0 0 0" />
-      <parent link="base_link" />
-      <child link="gyro_link" />
-    </joint>
-    <link name="gyro_link">
-    <inertial>
-      <mass value="0.001" />
-      <origin xyz="0 0 0" rpy="0 0 0" />
-      <inertia ixx="0.0001" ixy="0" ixz="0" iyy="0.000001" iyz="0" izz="0.0001" />
-    </inertial>
-    </link>
     <!-- Simulation sensors -->
     <xacro:sim_create_base/>
     <xacro:sim_create_wall_sensor/>
     <xacro:sim_create_cliff_sensors/>
-    <xacro:sim_imu/>
   </xacro:macro>
 </robot>
